File: Sanji V1/Sanji V1.kicad_pcb (KiCad board)
At the start: 2 copper layers, 85.5 x 40 mm, 64 parts, among them J1 Conn_01x03_Pin, J10 Conn_01x03_Pin, J11 Conn_01x03_Pin, J12 Conn_01x03_Pin, J2 INICIO, J3 DISPLAY, J4 Conn_01x03_Pin, J6 Conn_01x03_Pin, J7 Conn_01x03_Pin, J8 Conn_01x03_Pin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

Commit message: Add files via upload
Parts:
- added G***: LOGO, LOGO, F.Cu at (142.8, 103.2)
- added G***: LOGO, LOGO, B.Cu at (168.8, 103.0)
- added G***: LOGO, LOGO, B.Cu at (112.0, 101.4)
- added G***: LOGO, LOGO, B.Cu at (139.9, 105.4)
- J2: value INICIO -> Conn_01x03_Pin
- SW1, SW2, SW5, SW6: footprint Button_Switch_SMD:SW_Tactile_SPST_NO_Straight_CK_PTS636Sx25SMTRLFS -> BTN_SMD 3X6X3,5:SW_RS-032G05A3-SMRT
- moved R5 1.50 mm to (174.5, 101.0)
- moved R8 1.30 mm to (172.5, 101.0)
- moved R15 0.85 mm to (117.0, 96.4)
- moved R17 0.85 mm to (119.2, 96.4)
Routing:
- net VCC1: track 34.0 -> 0.00 mm, vias 1 -> 0
- net +5V: track 9.00 -> 5.35 mm, vias 10 -> 9
- net Net-(J6-Pin_3): track 7.64 -> 8.99 mm
- net /SCL: track 57.9 -> 58.4 mm
- net 3V3: vias 2 -> 6
- net /M2: vias 0 -> 1
- net /M1: vias 0 -> 1
- added copper zone on F.Cu, net VCC1
Other:
- board text added: "0V"
- board text added: "3V"
- board text added: "5V"
- board text added: "BT"
- board text added: "S"
- board text removed: "S1"
- board text removed: "S2"
- board text removed: "S3"
- board text removed: "S4"
- board text removed: "S5"
- board text removed: "S6"
- board text removed: "S7"
