File: Sanji V1/Sanji V1.kicad_sch (KiCad schematic)
At the start: 64 parts, among them J1 Conn_01x03_Pin, J10 Conn_01x03_Pin, J11 Conn_01x03_Pin, J12 Conn_01x03_Pin, J2 INICIO, J3 DISPLAY, J4 Conn_01x03_Pin, J6 Conn_01x03_Pin, J7 Conn_01x03_Pin, J8 Conn_01x03_Pin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

Commit message: Add files via upload
Parts:
- J2: value INICIO -> Conn_01x03_Pin
- SW1, SW2, SW5, SW6: footprint Button_Switch_SMD:SW_Tactile_SPST_NO_Straight_CK_PTS636Sx25SMTRLFS -> BTN_SMD 3X6X3,5:SW_RS-032G05A3-SMRT
Other:
- moved on the sheet: J10, J11, J4, J6, J7, J8, J9
